File: TimeMachine.kicad_pcb (KiCad board)
At the start: 4 copper layers, 107.6 x 59.8 mm, 51 parts, among them J1 AppleIIBus, J2 JTAG, U1 EPM7128SL84, U2 DS1315S-5, U3 74AHCT04, U4 AS6C8008, U5 39F040, Y1 32k768

Commit message: Regenerated gerbers
Other:
- board text added: "TimeMachine"
- board text removed: "4205A"
- board text removed: "GW"
Changed lines of the file:
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@@
   (general
     (thickness 1.6)
-    (drawings 38)
+    (drawings 37)
     (tracks 1947)
     (zones 0)
@@
     (effects (font (size 0.8128 0.8128) (thickness 0.2032)) (justify mirror))
   )
-  (gr_text GW (at 154.178 129.032) (layer F.SilkS)
+  (gr_text TimeMachine (at 156.972 129.032) (layer F.SilkS)
     (effects (font (size 1.524 1.524) (thickness 0.3)))
   )
@@
   (gr_arc (start 142.113 129.54) (end 139.573 129.54) (angle -90) (layer Edge.Cuts) (width 0.15))
   (gr_line (start 139.573 129.54) (end 139.573 96.139) (layer Edge.Cuts) (width 0.15))
-  (gr_text 4205A (at 159.766 129.032) (layer F.SilkS)
-    (effects (font (size 1.524 1.524) (thickness 0.3)))
-  )
   (gr_line (start 175.514 132.08) (end 175.514 139.192) (layer Edge.Cuts) (width 0.15))
   (gr_poly (pts (xy 241.3 139.446) (xy 240.792 139.954) (xy 175.768 139.954) (xy 175.26 139.446) (xy 175.26 132.08) (xy 241.3 132.08)) (layer B.Mask) (width 0))
