File: TimeMachine.kicad_sch (KiCad schematic)
At the start: 53 parts, among them J1 AppleIIBus, J2 JTAG, SW1 Mode, U1 EPM7128SL84, U2 DS1315S-5, U3 74AHCT04, U4 AS6C8008, U5 39F040, Y1 32k768

Commit message: Newer
Parts:
- removed C10, C11, C13, C17: DNP, stdpads:CP_EIA-3528, symbol Device:CP_Small
- removed C20, C24, C25: DNP, stdpads:C_0805, symbol Device:C_Small
- removed JP2: Clock, Connector_PinHeader_2.54mm:PinHeader_1x02_P2.54mm_Vertical_SMD_Pin1Left, symbol Device:Jumper_NO_Small
- added C10, C13, C17: 10u, stdpads:C_0805, symbol Device:C_Small
- added C11: 2u2, stdpads:C_0805, symbol Device:C_Small
- added R9: 100, stdpads:R_0805, symbol Device:R_Small
- added U6: XC6206P332MR, stdpads:SOT-23, symbol Regulator_Linear:XC6206PxxxMR
- H2, H3, H4, H5: footprint stdpads:PasteHole_1.1mm_PTH -> stdpads:PasteHole_1.152mm_NPTH; symbol Mechanical:MountingHole_Pad -> Mechanical:MountingHole
- R6: value 15 -> 1k
- R7: value 22k -> DNP
- R8: value 1k -> 0
Connections:
- net +5C: now also C17.1
- net +5V: now also C11.1, U6.3 (VI); no longer C8.1, U3.14 (VCC)
- net +BATT: now also C10.1
- net A2: now also SW1.1
- net DS~{WE}: now also SW1.4
- net GND: now also C10.2, C11.2, C13.2, C17.2, U6.1 (GND); no longer H2.1, H3.1, H4.1, H5.1, R8.1
- net RA1: no longer R7.1, SW1.1
- net RAMROMCSgb: now also R9.2; no longer U3.6
- net +3V3: now reaches R8.2
- net +3V3: now also C13.1, U6.2 (VO); no longer SW1.4
- new net: R9.1, U3.6
- new net V04: C8.1, R7.1, R8.1, U3.14 (VCC)
Other:
- moved on the sheet: BT1, C26, C8, C9, H1, R2, R4, R6, U2, U3C, Y1

Commit message: idk
Parts:
- removed J2: JTAG, stdpads:IDC_SMD_2x05_P2.54mm_Vertical, symbol Connector_Generic:Conn_02x05_Odd_Even
- added C20, C22, C27, C28: 2u2, stdpads:C_0805, symbol Device:C_Small
- added C23, C24: 22p, stdpads:C_0603, symbol Device:C_Small
- added C25: 100n, stdpads:C_0603, symbol Device:C_Small
- added J2: microUSB, stdpads:USB_Micro-B_ShouHan_MicroXNJ, symbol Connector:USB_B_Micro
- added R10, R11: 10k, stdpads:R_0805, symbol Device:R_Small
- added R12: 15, stdpads:R_0805, symbol Device:R_Small
- added U7: CH340G, stdpads:SOIC-16_3.9mm, symbol Interface_USB:CH340G
- added Y2: 12M, stdpads:Crystal_SMD_3225-4Pin_3.2x2.5mm, symbol Device:Crystal_GND24_Small
Connections:
- net +3V3: now also U7.10 (~{DSR}), U7.11 (~{RI})
- net +5V: now also C20.1, C22.1, C27.1, R10.1, U7.16 (VCC)
- net GND: now also C20.2, C22.2, C23.2, C24.2, C25.2, C27.2, C28.2, J2.5 (GND), J2.6 (Shield), R11.2, U7.1 (GND), Y2.2, Y2.4
- net TCK: now also R12.2
- net TDI: now also U7.13 (~{DTR})
- net TDO: now also U7.9 (~{CTS})
- net TMS: now also U7.14 (~{RTS})
- new net: J2.2 (D-), U7.6 (UD-)
- new net: J2.3 (D+), U7.5 (UD+)
- new net: R12.1, U7.2 (TXD)
- new net: R11.1, U7.15 (R232)
- new net: R10.2, U7.3 (RXD)
- new net: C24.1, U7.7 (XI), Y2.1
- new net: C23.1, U7.8 (XO), Y2.3
- new net CH340G3V3: C25.1, U7.4 (V3)
- new net USB5V: C28.1, J2.1 (VBUS)
- no-connect marks 6 -> 5
Other:
- moved on the sheet: BT1, C18, C8, R2, R4, R5, R6, R9, SW1, U2, U3A, U3B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
