File: Bus.kicad_sch (KiCad schematic)
At the start: 14 parts, among them J1 AppleIIBus, Q1 MMBT3904, Q2 MMBT3904, U4 74AHC245PW, U5 74AHC245PW, U6 74AHC245PW, U9 74AHC245PW

Commit message: Start on hibernate
Connections:
- net GND: no longer U4.8 (A6), U4.9 (A7)
- net B~{POR}: now reaches U4.11 (B7)
- new net ~{POR}: U4.9 (A7)
- no-connect marks 2 -> 1
Changed lines of the file:
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@@
 (kicad_sch (version 20230121) (generator eeschema)
   (paper "A4")
-  (junction (at 86.36 43.18) (diameter 0) (color 0 0 0 0)
-  )
   (junction (at 45.72 162.56) (diameter 0) (color 0 0 0 0)
   )
-  (junction (at 86.36 40.64) (diameter 0) (color 0 0 0 0)
-  )
   (junction (at 64.77 187.96) (diameter 0) (color 0 0 0 0)
   )
@@
   )
   (no_connect (at 106.68 40.64))
-  (no_connect (at 106.68 43.18))
   (bus_entry (at 76.2 124.46) (size 2.54 2.54)
     (stroke (width 0) (type default))
@@
     (stroke (width 0) (type default))
   )
-  (wire (pts (xy 86.36 38.1) (xy 86.36 40.64))
-    (stroke (width 0) (type default))
-  )
   (wire (pts (xy 106.68 86.36) (xy 114.3 86.36))
     (stroke (width 0) (type default))
@@
     (stroke (width 0) (type default))
   )
-  (wire (pts (xy 86.36 40.64) (xy 86.36 43.18))
-    (stroke (width 0) (type default))
-  )
   (wire (pts (xy 48.26 93.98) (xy 53.34 93.98))
     (stroke (width 0) (type default))
@@
   (label "BD2" (at 106.68 121.92 0) (fields_autoplaced)
     (effects (font (size 1.27 1.27)) (justify left bottom))
+  )
+  (hierarchical_label "~{POR}" (shape input) (at 86.36 40.64 180) (fields_autoplaced)
+    (effects (font (size 1.27 1.27)) (justify right))
   )
   (hierarchical_label "D~{OE}" (shape input) (at 106.68 114.3 0) (fields_autoplaced)
@@
     (effects (font (size 1.27 1.27)) (justify left))
   )
+  (hierarchical_label "B~{POR}" (shape output) (at 106.68 43.18 0) (fields_autoplaced)
+    (effects (font (size 1.27 1.27)) (justify left))
+  )
