File: TimeDisk.kicad_pcb (KiCad board)
At the start: 4 copper layers, 107.6 x 59.8 mm, 76 parts, among them J1 AppleIIBus, J2 microUSB, SW1 Mode, U1 EPM7128SL84, U2 DS1315S-5, U3 74LVC04AD, U4 AS6C8008, U5 39F040, U6 XC6206P332MR, U7 CH340G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

Commit message: idk if it's even good
Connections:
- C25 pad 1: CH340G3V3 -> +3V3
- C27 pad 1: +5V -> +3V3
- U7 pad 16: +5V -> +3V3
- U7 pad 4: CH340G3V3 -> +3V3
Routing:
- net +3V3: track 50.8 -> 172.7 mm, vias 2 -> 7
- net +5V: track 113.7 -> 107.7 mm, vias 63 -> 59
- net CH340G3V3: track 1.97 -> 0.00 mm
- net /ID2: track 16.8 -> 17.7 mm
- net /C~{RES}: track 148.1 -> 148.7 mm, vias 2 -> 4

Commit message: Done?
Parts:
- removed R11, R13, R18, R20: 22k, stdpads:R_0805
- removed R17, R19, R21: DNP, stdpads:R_0805
- added R1: DNP, stdpads:R_0805, F.Cu at (243.9, 119.1)
- added R3: 1k, stdpads:R_0805, F.Cu at (241.8, 119.1)
Connections:
- C25 pad 1: +3V3 -> /CH340_3V3
- C27 pad 1: +3V3 -> +5V
- U7 pad 10: /ID0 -> +5V
- U7 pad 11: /ID1 -> +5V
- U7 pad 12: /ID2 -> /~{DCD}
- U7 pad 15: Net-(U7-R232) -> GND
- U7 pad 16: +3V3 -> +5V
- U7 pad 4: +3V3 -> /CH340_3V3
Routing:
- net +3V3: track 172.7 -> 54.0 mm, vias 7 -> 2
- net /ID1: track 20.1 -> 0.00 mm, vias 2 -> 0
- net /~{DCD}: track 0.00 -> 18.4 mm, vias 0 -> 2
- net /ID2: track 17.7 -> 0.00 mm, vias 2 -> 0
- net /ID0: track 14.1 -> 0.00 mm, vias 2 -> 0
- net Net-(U7-R232): track 9.19 -> 0.00 mm
- net +5V: track 107.7 -> 115.7 mm, vias 59 -> 64
- net Net-(J2-D+): track 42.5 -> 40.3 mm
- net Net-(J2-D-): track 42.4 -> 40.2 mm
- net /CH340_3V3: track 0.00 -> 1.97 mm
- net GND: track 184.4 -> 182.7 mm, vias 481 -> 480
- net /C~{RES}: track 148.7 -> 148.1 mm, vias 4 -> 2

Commit message: As sent to JLC
Parts:
- added J3: JTAG, stdpads:Header_2x5_Unshrouded_P1.27mm, B.Cu at (239.8, 99.8)
- added R11: 22k, stdpads:R_0805, F.Cu at (192.0, 97.6)
- added R13: 22k, stdpads:R_0805, F.Cu at (235.1, 122.7)
- moved C23 0.15 mm to (242.9, 105.9)
- turned U9 to 180 degrees
Connections:
- net Net-(U7-TXD) renamed /TCKr
Routing:
- net /TMS: track 20.2 -> 57.5 mm, vias 0 -> 3
- net /TDO: track 55.4 -> 75.9 mm, vias 2 -> 3
- net /TDI: track 6.54 -> 26.3 mm, vias 0 -> 1
- net /TCKr: track 13.4 -> 33.0 mm, vias 0 -> 1
- net /TCK: track 41.9 -> 50.5 mm
- net GND: track 182.7 -> 187.2 mm, vias 480 -> 487
- net /IRQ~{OE}: track 89.3 -> 93.6 mm
- net +5V: track 115.7 -> 119.1 mm, vias 64 -> 65
Other:
- board text added: "B10"

Commit message: Add RPP
Parts:
- added D1: 1N5819, stdpads:D_SOD-123, F.Cu at (147.2, 108.2)
- added D2: 1N5819, stdpads:D_SOD-123, F.Cu at (144.2, 112.3)
- added D3: 10V, stdpads:D_SOD-323, F.Cu at (142.7, 108.2)
- added Q1: AO3401A, stdpads:SOT-23, F.Cu at (142.7, 105.2)
- added R14: 220, stdpads:R_0805, F.Cu at (142.6, 110.2)
- added R17: 220, stdpads:R_0805, F.Cu at (142.7, 101.5)
- moved C10 7.18 mm to (148.7, 111.8), turned to 180 degrees
Connections:
- BT1 pad 1: +BATT -> Net-(BT1-+)
- U3 pad 7: GND -> unconnected-(U3G-GND-Pad7)
Routing:
- net Net-(BT1-+): track 0.00 -> 125.2 mm, vias 0 -> 6
- net +BATT: track 180.9 -> 57.3 mm, vias 11 -> 7
- net Net-(D1-A): track 0.00 -> 10.2 mm
- net Net-(D3-A): track 0.00 -> 4.01 mm
- net GND: track 187.2 -> 189.2 mm, vias 487 -> 483
Other:
- board text added: "B11"
- board text removed: "B10"
