File: TimeDisk.kicad_pcb (KiCad board)
At the start: 4 copper layers, 107.6 x 59.8 mm, 77 parts, among them J1 AppleIIBus, J2 microUSB, J3 JTAG, Q1 AO3401A, SW1 Mode, U1 EPM7128SL84, U2 DS1315S-5, U3 74LVC04AD, U4 AS6C8008, U5 39F040, U6 XC6206P332MR, U7 CH340G, U8 74LVC1G74DC, U9 74AHCT1G125GW, Y1 32k768, Y2 12M

Commit message: Go back to calling this version 1.0... RC 1.0
Other:
- board text added: "B10"
- board text removed: "B11"
Changed lines of the file:
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@@
     (effects (font (size 1.27 1.27) (thickness 0.2)) (justify mirror))
   )
-  (gr_text "B11" (at 230.0605 129.921) (layer "B.SilkS")
+  (gr_text "B10" (at 230.0605 129.921) (layer "B.SilkS")
     (effects (font (size 0.8128 0.8128) (thickness 0.2032)) (justify mirror))
   )

Commit message: idk
Parts:
- removed R10: 22k, stdpads:R_0805
- R14, R17: value 220 -> 600
- Y1: footprint Crystal:Crystal_C26-LF_D2.1mm_L6.5mm_Horizontal -> stdpads:Crystal_C26-LF_D2.1mm_L6.5mm_Horizontal
- moved R17 10.6 mm to (151.4, 107.6), turned to 0 degrees
- moved FID3 5.27 mm to (161.1, 82.4)
- moved H3 5.27 mm to (163.6, 82.4)
- moved FID2 4.83 mm to (142.1, 101.0)
- moved BT1 2.69 mm to (153.8, 94.1)
- moved H2 0.63 mm to (141.7, 98.2)
- moved D1 0.60 mm to (147.2, 107.6)
- moved D3 0.60 mm to (142.7, 107.6)
- moved Q1 0.60 mm to (142.7, 104.6)
- moved R14 0.60 mm to (142.6, 109.6)
- moved D2 0.60 mm to (144.2, 111.8)
Connections:
- U7 pad 3: Net-(U7-RXD) -> +5V
Routing:
- net Net-(U7-RXD): track 8.66 -> 0.00 mm, vias 2 -> 0
- net Net-(BT1-+): track 120.0 -> 128.6 mm, vias 6 -> 7
- net GND: track 187.8 -> 189.0 mm, vias 488 -> 492
- net +BATT: track 57.3 -> 58.2 mm
Other:
- board text removed: "Positive Up"

Commit message: RC
Parts:
- removed the R6 at (233.8, 126.7)
- removed the R7 at (169.8, 111.3)
- removed the R8 at (169.8, 109.2)
- C10, C12, C13, C14, C15, C16, C17, C29, C8: value 10u -> 2u2
- R1: renamed from R4; value 22k -> 4k7
- moved C29 0.55 mm to (191.1, 83.8)
- moved R6 0.55 mm to (194.8, 83.8)
- moved U8 0.55 mm to (191.3, 87.7)
- renumbered R13 to R10, R5 to R3, R9 to R4, R12 to R5, R16 to R6, R17 to R7, R14 to R8, R11 to R9
Connections:
- C8 pad 1: /V04 -> +3V3
- U2 pad 13: /C~{RES} -> /~{RES}
- U3 pad 14: /V04 -> +3V3
Routing:
- net /C~{RES}: track 148.4 -> 0.00 mm, vias 2 -> 0
- net /~{RES}: track 36.7 -> 183.9 mm
- net +3V3: track 82.7 -> 89.2 mm
- net /V04: track 6.35 -> 0.00 mm
- net /D0: track 67.9 -> 64.2 mm
- net +12V: track 34.9 -> 32.7 mm
- net +5V: track 120.0 -> 121.5 mm, vias 65 -> 66
- net +5C: track 76.1 -> 74.6 mm
- net GND: track 189.0 -> 190.4 mm, vias 492 -> 501
- net /RA0: track 23.2 -> 22.2 mm
- net /RAMCS: track 42.9 -> 41.9 mm
- net /IRQ~{OE}: track 89.8 -> 90.3 mm
