File: Docs.kicad_sch (KiCad schematic)
At the start: 0 parts

Commit message: with hole
Other:
- title: Time Machine -> GW4206B (TimeDisk)
Changed lines of the file:
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@@
   (paper "USLetter")
   (title_block
-    (title "Time Machine")
-    (date "2019-10-13")
-    (rev "0.9")
+    (title "GW4206B (TimeDisk)")
+    (date "2024-03-21")
+    (rev "1.1")
     (company "Garrett's Workshop")
   )

Commit message: RC
Other:
- note removed: "6502-Accessible Registers"
- note removed: "Addr[19:16] = (S6 & AddrHSEL & ~{R}W) ? D[3:0] : Addr[19:16] @ C7M Addr[15:8] = (S6 if AddrMSEL & ~{R}W) ? D[7:0] : Addr[15:8] @ C7M Addr[7:0] = (S6 if AddrLSEL & ~{R}W) ? D[7:0] : Addr[7:0] @ C7M if (RAMSEL & S1) Addr[19:0]++ @ C7M Bank[7:0] = (S6 & BankSEL & ~{R}W) ? D[7:0] : Bank[7:0] @ C7M"
- note removed: "Address Bus Routing"
- note removed: "BankSEL = S3 ? (A==XXXF & DEVSEL & REGEN) : BankSEL @ C7M RAMSEL = S3 ? (A==XXX3 & DEVSEL & REGEN) : RAMSEL @ C7M AddrHSEL = S3 ? (A==XXX2 & DEVSEL & REGEN) : AddrHSEL @ C7M AddrMSEL = S3 ? (A==XXX1 & DEVSEL & REGEN) : AddrMSEL @ C7M AddrLSEL = S3 ? (A==XXX0 & DEVSEL & REGEN) : AddrLSEL @ C7M REGEN = (IOSEL & S3) ? 1 : REGEN @ C7M IOROMEN = (A==XXFF & IOSTRB & S3) ? 0 : (A==XX00 & IOSEL & S3) ? 1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"
- note removed: "DBEN = ~{S2} @ C7M RAMROMCS = RAMSEL | IOSEL | (IOSTRB & IOROMEN) RAMCS = RAMSEL ROMCS = RAMROMCSgb & (IOSEL | (IOSTRB & IOROMEN))"
- note removed: "Data Bus Routing"
- note removed: "Information here may be out of date, superseded by ./cpld/TimeMachine.v"
- note removed: "PHI0reg = PHI0 @ C7M S[3:0] = (~{PHI0} & PHI0reg) ? 1 : (S==0) ? 0 : S+1 @ C7M"
- note removed: "RA[19] = Addr[19] RA[18:12] = RAMSEL ? Addr[18:12] : Bank[6:0] RA[11] = RAMSEL ? Addr[18:12] : A[11] RA[10:0] = Addr[11:0]"
- note removed: "RD[7:0] = (~{DEVSEL} | R~{W}) ? 8’bZ : D[7:0] D[7:0] = (~{CSEN} | ~{DEVSEL} | ~{R}W) ? 8’bZ : AddrHSEL ? {4’hF, Addr[22:16]} : AddrMSEL ? Addr[15:8] : AddrLSEL ? Addr[7:0] : RD[7:0]"
- note removed: "ROM / SRAM Control"
- note removed: "Select signals (registered)"
- note removed: "State Synchronization"
- title: GW4206B (TimeDisk) -> TimeDisk (GW4206B)
Changed lines of the file:
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@@
   (paper "USLetter")
   (title_block
-    (title "GW4206B (TimeDisk)")
-    (date "2024-03-21")
-    (rev "1.1")
+    (title "TimeDisk (GW4206B)")
+    (date "2024-04-23")
+    (rev "1.0")
     (company "Garrett's Workshop")
   )
@@
   (bus (pts (xy 124.46 24.13) (xy 124.46 40.64))
     (stroke (width 0) (type default))
-  )
-  (text "ROM / SRAM Control" (at 109.22 72.39 0)
-    (effects (font (size 2.54 2.54)) (justify left bottom))
   )
   (text "S7" (at 38.1 27.94 0)
@@
     (effects (font (size 1.016 1.016)) (justify left bottom))
   )
-  (text "Data Bus Routing" (at 181.61 105.41 0)
-    (effects (font (size 2.54 2.54)) (justify left bottom))
-  )
-  (text "PHI0reg = PHI0 @ C7M\nS[3:0] = (~{PHI0} & PHI0reg) ? 1 : \n          (S==0) ? 0 : S+1 @ C7M"
-    (at 34.29 78.74 0)
-    (effects (font (size 1.27 1.27)) (justify left bottom))
-  )
-  (text "RD[7:0] = (~{DEVSEL} | R~{W}) ? 8’bZ : D[7:0]\nD[7:0] = (~{CSEN} | ~{DEVSEL} | ~{R}W) ? 8’bZ :\n          AddrHSEL ? {4’hF, Addr[22:16]} : \n          AddrMSEL ? Addr[15:8] : \n          AddrLSEL ? Addr[7:0] :\n          RD[7:0]"
-    (at 182.88 119.38 0)
-    (effects (font (size 1.27 1.27)) (justify left bottom))
-  )
   (text "S2" (at 190.5 27.94 0)
     (effects (font (size 1.016 1.016)) (justify left bottom))
@@
     (effects (font (size 1.016 1.016)) (justify left bottom))
   )
-  (text "Addr[19:16] = (S6 & AddrHSEL & ~{R}W) ? D[3:0] : Addr[19:16] @ C7M\nAddr[15:8] = (S6 if AddrMSEL & ~{R}W) ? D[7:0] : Addr[15:8] @ C7M\nAddr[7:0] = (S6 if AddrLSEL & ~{R}W) ? D[7:0] : Addr[7:0] @ C7M\nif (RAMSEL & S1) Addr[19:0]++ @ C7M\nBank[7:0] = (S6 & BankSEL & ~{R}W) ? D[7:0] : Bank[7:0] @ C7M"
-    (at 182.88 99.06 0)
-    (effects (font (size 1.27 1.27)) (justify left bottom))
-  )
   (text "S2" (at 68.58 27.94 0)
     (effects (font (size 1.016 1.016)) (justify left bottom))
@@
     (effects (font (size 1.016 1.016)) (justify left bottom))
   )
-  (text "State Synchronization" (at 33.02 72.39 0)
-    (effects (font (size 2.54 2.54)) (justify left bottom))
-  )
   (text "Video Access" (at 167.64 21.59 0)
     (effects (font (size 2.6416 2.6416)) (justify left bottom))
   )
-  (text "6502-Accessible Registers" (at 181.61 87.63 0)
-    (effects (font (size 2.54 2.54)) (justify left bottom))
-  )
   (text "6502 CPU Access" (at 218.44 21.59 0)
     (effects (font (size 2.54 2.54)) (justify left bottom))
   )
-  (text "Address Bus Routing" (at 181.61 72.39 0)
-    (effects (font (size 2.54 2.54)) (justify left bottom))
-  )
   (text "S5" (at 236.22 27.94 0)
     (effects (font (size 1.016 1.016)) (justify left bottom))
@@
   (text "S5" (at 114.3 27.94 0)
     (effects (font (size 1.016 1.016)) (justify left bottom))
-  )
-  (text "RA[19] = Addr[19]\nRA[18:12] = RAMSEL ? Addr[18:12] : Bank[6:0]\nRA[11] = RAMSEL ? Addr[18:12] : A[11]\nRA[10:0] = Addr[11:0]"
-    (at 182.88 81.28 0)
-    (effects (font (size 1.27 1.27)) (justify left bottom))
-  )
-  (text "BankSEL = S3 ? (A==XXXF & DEVSEL & REGEN) : BankSEL @ C7M\nRAMSEL = S3 ? (A==XXX3 & DEVSEL & REGEN) : RAMSEL @ C7M\nAddrHSEL = S3 ? (A==XXX2 & DEVSEL & REGEN) : AddrHSEL @ C7M\nAddrMSEL = S3 ? (A==XXX1 & DEVSEL & REGEN) : AddrMSEL @ C7M\nAddrLSEL = S3 ? (A==XXX0 & DEVSEL & REGEN) : AddrLSEL @ C7M\n\nREGEN = (IOSEL & S3) ? 1 : REGEN @ C7M\nIOROMEN = (A==XXFF & IOSTRB & S3) ? 0 :\n            (A==XX00 & IOSEL & S3) ? 1 :\n            IOROMEN @ C7M"
-    (at 34.29 106.68 0)
-    (effects (font (size 1.27 1.27)) (justify left bottom))
   )
   (text "Video Access" (at 45.72 21.59 0)
@@
     (effects (font (size 1.27 1.27)) (justify right bottom))
   )
-  (text "Select signals (registered)" (at 33.02 85.09 0)
-    (effects (font (size 2.54 2.54)) (justify left bottom))
-  )
-  (text "DBEN = ~{S2} @ C7M\n\nRAMROMCS = RAMSEL | IOSEL | (IOSTRB & IOROMEN)\nRAMCS = RAMSEL\nROMCS = RAMROMCSgb & (IOSEL | (IOSTRB & IOROMEN))"
-    (at 110.49 83.82 0)
-    (effects (font (size 1.27 1.27)) (justify left bottom))
-  )
-  (text "Information here may be out of date,\nsuperseded by ./cpld/TimeMachine.v"
-    (at 35.56 140.97 0)
-    (effects (font (size 5.08 5.08)) (justify left bottom))
-  )
   (text "S6" (at 129.54 27.94 0)
