File: TimeDisk.kicad_sch (KiCad schematic)
At the start: 75 parts, among them J1 AppleIIBus, J2 microUSB, J3 JTAG, Q1 AO3401A, SW1 Mode, U1 EPM7128SL84, U2 DS1315S-5, U3 74LVC04AD, U4 AS6C8008, U5 39F040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

Commit message: idk
Parts:
- removed R10: 22k, stdpads:R_0805, symbol Device:R_Small
- R14, R17: value 220 -> 600
- Y1: footprint Crystal:Crystal_C26-LF_D2.1mm_L6.5mm_Horizontal -> stdpads:Crystal_C26-LF_D2.1mm_L6.5mm_Horizontal
Connections:
- net +5V: now also U7.3 (RXD)
Changed lines of the file:
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@@
     (stroke (width 0) (type default))
   )
-  (wire (pts (xy 189.23 27.94) (xy 189.23 33.02))
-    (stroke (width 0) (type default))
-  )
   (bus (pts (xy 124.46 119.38) (xy 124.46 121.92))
     (stroke (width 0) (type default))
@@
     (stroke (width 0) (type default))
   )
+  (wire (pts (xy 189.23 22.86) (xy 189.23 33.02))
+    (stroke (width 0) (type default))
+  )
   (wire (pts (xy 234.95 83.82) (xy 234.95 74.93))
     (stroke (width 0) (type default))
@@
       (effects (font (size 1.27 1.27)) (justify left))
     )
-    (property "Footprint" "Crystal:Crystal_C26-LF_D2.1mm_L6.5mm_Horizontal" (at 232.41 106.68 0)
+    (property "Footprint" "stdpads:Crystal_C26-LF_D2.1mm_L6.5mm_Horizontal" (at 232.41 106.68 0)
       (effects (font (size 1.27 1.27)) hide)
     )
@@
       (effects (font (size 1.27 1.27)) (justify right))
     )
-    (property "Value" "220" (at 248.92 88.9 0)
+    (property "Value" "600" (at 248.92 88.9 0)
       (effects (font (size 1.27 1.27)) (justify right))
     )
@@
     )
   )
-  (symbol (lib_id "Device:R_Small") (at 189.23 25.4 0) (unit 1)
-    (in_bom yes) (on_board yes) (dnp no)
-    (property "Reference" "R10" (at 187.96 24.13 0)
-      (effects (font (size 1.27 1.27)) (justify right))
-    )
-    (property "Value" "22k" (at 187.96 26.67 0)
-      (effects (font (size 1.27 1.27)) (justify right))
-    )
-    (property "Footprint" "stdpads:R_0805" (at 189.23 25.4 0)
-      (effects (font (size 1.27 1.27)) hide)
-    )
-    (property "Datasheet" "~" (at 189.23 25.4 0)
-      (effects (font (size 1.27 1.27)) hide)
-    )
-    (property "LCSC Part" "C25804" (at 189.23 25.4 0)
-      (effects (font (size 1.27 1.27)) hide)
-    )
-    (pin "1")
-    (pin "2")
-    (instances
-      (project "TimeDisk"
-        (path "/4fa10683-33cd-4dcd-8acc-2415cd63c62a"
-          (reference "R10") (unit 1)
-        )
-      )
-    )
-  )
   (symbol (lib_id "power:+3V3") (at 205.74 68.58 0) (unit 1)
     (in_bom yes) (on_board yes) (dnp no)
@@
       (effects (font (size 1.27 1.27)) (justify top))
     )
-    (property "Value" "220" (at 256.54 69.85 90)
+    (property "Value" "600" (at 256.54 69.85 90)
       (effects (font (size 1.27 1.27)) (justify bottom))
     )

Commit message: RC
Parts:
- removed R11, R13: DNP, stdpads:R_0805, symbol Device:R_Small
- removed R12, R16: 15, stdpads:R_0805, symbol Device:R_Small
- removed R14, R17: 600, stdpads:R_0805, symbol Device:R_Small
- added R1, R3: 4k7, stdpads:R_0805, symbol Device:R_Small
- added R10: DNP, stdpads:R_0805, symbol Device:R_Small
- C10, C12, C13, C14, C15, C16, C17, C29, C8: value 10u -> 2u2
- R4: value 22k -> 15
- R5: value 4k7 -> 15
- R6: value 1k -> 15
- R7: value DNP -> 600
- R8: value 0 -> 600
- R9: value 15 -> DNP
Connections:
- net +3V3: now also C8.1, U3.14 (VCC); no longer R8.2
- net +5V: now also R1.2, R10.1, R3.1; no longer R4.2, R5.1, R7.2
- net DS~{WE}: now also R1.1; no longer R4.1
- net GND: now also R8.1, R9.2
- net IRQ~{OE}: now also R6.1
- net RAMROMCSgb: now also R4.2; no longer R9.2
- net TCK: now also R5.2, R9.1
- net TCKr: now also R5.1
- net TMS: now also R10.2
- net ~{RES}: now also U2.13 (~{RST}); no longer R6.2
- net at U3.6: now also R4.1; no longer R9.1
- net at BT1.1 (+): now also R7.2
- net at D3.2 (A), Q1.1 (G): now also R8.2
- net at D1.2 (A), Q1.3 (D): now also R7.1
- net at SW1.3: now also R3.2; no longer R5.2
- net at U8.5 (Q): now also R6.2
- removed net C~{RES}: R6.1, U2.13 (~{RST})
- removed net V04: C8.1, R7.1, R8.1, U3.14 (VCC)

Commit message: RC
Parts:
- removed C30: 2u2, stdpads:C_0805, symbol Device:C_Small
- removed R6: 15, stdpads:R_0805, symbol Device:R_Small
- removed U9: 74AHCT1G125GW, stdpads:SOT-353, symbol GW_Logic:741G125GW
- C1, C10, C11, C12, C13, C14, C15, C16, C17, C18, C19, C2, C20, C21, C22, C26, C29, C3, C4, C5, C6, C7, C8, C9: LCSC Part (none) -> C87994
- C27, C28: LCSC Part C23630 -> C87994
- D1, D2: value 1N5819 -> 1N5819WS; LCSC Part C22452 -> C191023
- D3: LCSC Part C235983 -> C118604
- J2: LCSC Part C404969 -> C132564
- J3: Notes DNP - test pad connector -> (none)
- Q1: LCSC Part (none) -> C15127
- R1, R2, R3: LCSC Part (none) -> C17673
- R4, R5: value 15 -> 22; LCSC Part (none) -> C17561
- R7, R8: value 600 -> 680; LCSC Part (none) -> C17798
- U3: LCSC Part (none) -> C190764
- U4: LCSC Part (none) -> C1349342
- U5: LCSC Part (none) -> C645936
- U6: LCSC Part (none) -> C5446
- U8: value 74LVC1G74DC -> 74LVC1G74DP; LCSC Part (none) -> C458768
Connections:
- net RA0: now also U8.5 (Q); no longer U1.55 (I/O), U8.2 (D)
- net RA1: now also U1.55 (I/O), U8.2 (D); no longer U1.52 (I/O), U8.1 (CK)
- net RA2: now also U8.1 (CK)
- net ~{IRQ}: now also U1.52 (I/O)
Other:
- title: GW4206B (TimeDisk) -> TimeDisk (GW4206B)
- moved on the sheet: C20, C22, C26, C7, C8, C9, U8

Commit message: B.1.0 RC2/3
Parts:
- D1, D2: value 1N5819WS -> BAT54H
Changed lines of the file:
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@@
       (effects (font (size 1.27 1.27)) (justify left))
     )
-    (property "Value" "1N5819WS" (at 223.52 73.66 90)
+    (property "Value" "BAT54H" (at 223.52 73.66 90)
       (effects (font (size 1.27 1.27)) (justify left))
     )
@@
       (effects (font (size 1.27 1.27)) (justify bottom))
     )
-    (property "Value" "1N5819WS" (at 247.65 66.04 0)
-      (effects (font (size 1.27 1.27)))
-    )
+    (property "Value" "BAT54H" (at 247.65 66.04 0)
+      (effects (font (size 1.27 1.27)))
+    )
